Commit message: finished adding terrains

File: test.urdf (robot description, URDF)
Before this commit: robot pepe, 5 links, 4 joints
Links:
- removed link 12
- removed link 13
- added link 15, mass 0.036815199820519305; collision cylinder length=0.7455079360214598 radius=0.12537545126732408; visual cylinder length=0.7455079360214598 radius=0.12537545126732408
- added link 22, mass 2.109157485313338; collision cylinder length=1.9581136678606774 radius=0.5855454606463423; visual cylinder length=1.9581136678606774 radius=0.5855454606463423
- added link 23, mass 2.109157485313338; collision cylinder length=1.9581136678606774 radius=0.5855454606463423; visual cylinder length=1.9581136678606774 radius=0.5855454606463423
- added link 26, mass 2.109157485313338; collision cylinder length=1.9581136678606774 radius=0.5855454606463423; visual cylinder length=1.9581136678606774 radius=0.5855454606463423
- added link 27, mass 2.109157485313338; collision cylinder length=1.9581136678606774 radius=0.5855454606463423; visual cylinder length=1.9581136678606774 radius=0.5855454606463423
- added link 28, mass 2.109157485313338; collision cylinder length=1.9581136678606774 radius=0.5855454606463423; visual cylinder length=1.9581136678606774 radius=0.5855454606463423
- link 0: mass 0.08882193011447076 -> 0.0006266931023623138; geometry collision cylinder length=1.7800595899717475 radius=0.010586081919601642; visual cylinder length=1.7800595899717475 radius=0.010586081919601642
- link 11: mass 1.3629571017358157 -> 0.036815199820519305; geometry collision cylinder length=0.7455079360214598 radius=0.12537545126732408; visual cylinder length=0.7455079360214598 radius=0.12537545126732408
- link 24: mass 0.00927975494390793 -> 2.109157485313338; geometry collision cylinder length=1.9581136678606774 radius=0.5855454606463423; visual cylinder length=1.9581136678606774 radius=0.5855454606463423
Joints:
- removed joint 12_to_0
- removed joint 13_to_0
- removed joint 24_to_0
- added joint 15_to_0: type revolute, parent 0, child 15, origin xyz=0.9211911784477138 0.9999 0.22097220481951255 rpy=10.030140424100777 5.507066050751844 2.4867577634447517, axis 1 0 0, limit lower=3.1415 upper=-3.1415 effort=1 velocity=1
- added joint 22_to_11: type revolute, parent 11, child 22, origin xyz=0.5723003634453724 0.7343359490418989 0.004789470228331982 rpy=8.582294283103815 6.022524202784673 3.2204442206050974, axis 0 1 0, limit lower=3.1415 upper=-3.1415 effort=1 velocity=1
- added joint 23_to_11: type revolute, parent 11, child 23, origin xyz=0.5723003634453724 0.7343359490418989 0.004789470228331982 rpy=12.873441424655724 6.022524202784673 3.2204442206050974, axis 0 1 0, limit lower=3.1415 upper=-3.1415 effort=1 velocity=1
- added joint 24_to_11: type revolute, parent 11, child 24, origin xyz=0.5723003634453724 0.7343359490418989 0.004789470228331982 rpy=17.16458856620763 6.022524202784673 3.2204442206050974, axis 0 1 0, limit lower=3.1415 upper=-3.1415 effort=1 velocity=1
- added joint 26_to_15: type revolute, parent 15, child 26, origin xyz=0.5723003634453724 0.7343359490418989 0.004789470228331982 rpy=8.582294283103815 6.022524202784673 3.2204442206050974, axis 0 1 0, limit lower=3.1415 upper=-3.1415 effort=1 velocity=1
- added joint 27_to_15: type revolute, parent 15, child 27, origin xyz=0.5723003634453724 0.7343359490418989 0.004789470228331982 rpy=12.873441424655724 6.022524202784673 3.2204442206050974, axis 0 1 0, limit lower=3.1415 upper=-3.1415 effort=1 velocity=1
- added joint 28_to_15: type revolute, parent 15, child 28, origin xyz=0.5723003634453724 0.7343359490418989 0.004789470228331982 rpy=17.16458856620763 6.022524202784673 3.2204442206050974, axis 0 1 0, limit lower=3.1415 upper=-3.1415 effort=1 velocity=1
- joint 11_to_0: axis 0 0 1 -> 1 0 0; origin xyz=0.13758607675745194 0.9350807390271525 0.7734982986138889 rpy=1.1448832225386056 4.335027266637536 1.6623373384868418 -> xyz=0.9211911784477138 0.9999 0.22097220481951255 rpy=6.686760282733851 5.507066050751844 2.4867577634447517

Commit message: add summit detection and encouragement

File: test.urdf (robot description, URDF)
Before this commit: robot pepe, 3 links, 2 joints
Links:
- added link 23, mass 0.023047021486861805; collision cylinder length=0.6813966216120516 radius=0.10376060110043672; visual cylinder length=0.6813966216120516 radius=0.10376060110043672
- added link 24, mass 0.023047021486861805; collision cylinder length=0.6813966216120516 radius=0.10376060110043672; visual cylinder length=0.6813966216120516 radius=0.10376060110043672
- link 0: mass 0.11132000648939905 -> 0.12562601080153418; geometry collision cylinder length=0.9999 radius=0.19998000000000002; visual cylinder length=0.9999 radius=0.19998000000000002
- link 11: mass 0.12388386395529906 -> 0.023047021486861805; geometry collision cylinder length=0.6813966216120516 radius=0.10376060110043672; visual cylinder length=0.6813966216120516 radius=0.10376060110043672
- link 12: mass 0.12388386395529906 -> 0.023047021486861805; geometry collision cylinder length=0.6813966216120516 radius=0.10376060110043672; visual cylinder length=0.6813966216120516 radius=0.10376060110043672
Joints:
- added joint 23_to_0: type revolute, parent 0, child 23, origin xyz=0.0 0.0 0.6110374662090388 rpy=9.183625862202506 6.282556988648868 0.7699242783357677, axis 0 0 1, limit lower=3.1415 upper=-3.1415 effort=1 velocity=1
- added joint 24_to_0: type revolute, parent 0, child 24, origin xyz=0.0 0.0 0.6110374662090388 rpy=11.479532327753132 6.282556988648868 0.7699242783357677, axis 0 0 1, limit lower=3.1415 upper=-3.1415 effort=1 velocity=1
- joint 11_to_0: axis 0 1 0 -> 0 0 1; origin xyz=0.0 0.0 0.8281286133482968 rpy=7.738725271434994 5.587068316070371 5.388748733323181 -> xyz=0.0 0.0 0.6110374662090388 rpy=4.591812931101253 6.282556988648868 0.7699242783357677
- joint 12_to_0: axis 0 1 0 -> 0 0 1; origin xyz=0.0 0.0 0.8281286133482968 rpy=11.608087907152491 5.587068316070371 5.388748733323181 -> xyz=0.0 0.0 0.6110374662090388 rpy=6.88771939665188 6.282556988648868 0.7699242783357677

Commit message: added energy and efficiency

File: test.urdf (robot description, URDF)
Before this commit: robot pepe, 5 links, 4 joints
Links:
- removed link 12
- removed link 23
- removed link 24
- added link 111, mass 0.015105155920040988; collision cylinder length=0.9406222288547907 radius=0.07149572114075056; visual cylinder length=0.9406222288547907 radius=0.07149572114075056
- added link 121, mass 0.015105155920040988; collision cylinder length=0.9406222288547907 radius=0.07149572114075056; visual cylinder length=0.9406222288547907 radius=0.07149572114075056
- added link 212, mass 0.015105155920040988; collision cylinder length=0.9406222288547907 radius=0.07149572114075056; visual cylinder length=0.9406222288547907 radius=0.07149572114075056
- added link 215, mass 0.015105155920040988; collision cylinder length=0.9406222288547907 radius=0.07149572114075056; visual cylinder length=0.9406222288547907 radius=0.07149572114075056
- added link 218, mass 0.015105155920040988; collision cylinder length=0.9406222288547907 radius=0.07149572114075056; visual cylinder length=0.9406222288547907 radius=0.07149572114075056
- added link 22, mass 0.015105155920040988; collision cylinder length=0.9406222288547907 radius=0.07149572114075056; visual cylinder length=0.9406222288547907 radius=0.07149572114075056
- added link 222, mass 0.015105155920040988; collision cylinder length=0.9406222288547907 radius=0.07149572114075056; visual cylinder length=0.9406222288547907 radius=0.07149572114075056
- added link 225, mass 0.015105155920040988; collision cylinder length=0.9406222288547907 radius=0.07149572114075056; visual cylinder length=0.9406222288547907 radius=0.07149572114075056
- added link 228, mass 0.015105155920040988; collision cylinder length=0.9406222288547907 radius=0.07149572114075056; visual cylinder length=0.9406222288547907 radius=0.07149572114075056
- added link 25, mass 0.015105155920040988; collision cylinder length=0.9406222288547907 radius=0.07149572114075056; visual cylinder length=0.9406222288547907 radius=0.07149572114075056
- added link 28, mass 0.015105155920040988; collision cylinder length=0.9406222288547907 radius=0.07149572114075056; visual cylinder length=0.9406222288547907 radius=0.07149572114075056
- added link 310, mass 0.001966705087677275; collision cylinder length=0.8083900654294837 radius=0.027828141337028135; visual cylinder length=0.8083900654294837 radius=0.027828141337028135
- added link 313, mass 0.001966705087677275; collision cylinder length=0.8083900654294837 radius=0.027828141337028135; visual cylinder length=0.8083900654294837 radius=0.027828141337028135
- added link 314, mass 0.001966705087677275; collision cylinder length=0.8083900654294837 radius=0.027828141337028135; visual cylinder length=0.8083900654294837 radius=0.027828141337028135
- added link 316, mass 0.001966705087677275; collision cylinder length=0.8083900654294837 radius=0.027828141337028135; visual cylinder length=0.8083900654294837 radius=0.027828141337028135
- added link 317, mass 0.001966705087677275; collision cylinder length=0.8083900654294837 radius=0.027828141337028135; visual cylinder length=0.8083900654294837 radius=0.027828141337028135
- added link 319, mass 0.001966705087677275; collision cylinder length=0.8083900654294837 radius=0.027828141337028135; visual cylinder length=0.8083900654294837 radius=0.027828141337028135
- added link 320, mass 0.001966705087677275; collision cylinder length=0.8083900654294837 radius=0.027828141337028135; visual cylinder length=0.8083900654294837 radius=0.027828141337028135
- added link 323, mass 0.001966705087677275; collision cylinder length=0.8083900654294837 radius=0.027828141337028135; visual cylinder length=0.8083900654294837 radius=0.027828141337028135
- added link 324, mass 0.001966705087677275; collision cylinder length=0.8083900654294837 radius=0.027828141337028135; visual cylinder length=0.8083900654294837 radius=0.027828141337028135
- added link 326, mass 0.001966705087677275; collision cylinder length=0.8083900654294837 radius=0.027828141337028135; visual cylinder length=0.8083900654294837 radius=0.027828141337028135
- added link 327, mass 0.001966705087677275; collision cylinder length=0.8083900654294837 radius=0.027828141337028135; visual cylinder length=0.8083900654294837 radius=0.027828141337028135
- added link 329, mass 0.001966705087677275; collision cylinder length=0.8083900654294837 radius=0.027828141337028135; visual cylinder length=0.8083900654294837 radius=0.027828141337028135
- added link 33, mass 0.001966705087677275; collision cylinder length=0.8083900654294837 radius=0.027828141337028135; visual cylinder length=0.8083900654294837 radius=0.027828141337028135
- added link 330, mass 0.001966705087677275; collision cylinder length=0.8083900654294837 radius=0.027828141337028135; visual cylinder length=0.8083900654294837 radius=0.027828141337028135
- added link 34, mass 0.001966705087677275; collision cylinder length=0.8083900654294837 radius=0.027828141337028135; visual cylinder length=0.8083900654294837 radius=0.027828141337028135
- added link 36, mass 0.001966705087677275; collision cylinder length=0.8083900654294837 radius=0.027828141337028135; visual cylinder length=0.8083900654294837 radius=0.027828141337028135
- added link 37, mass 0.001966705087677275; collision cylinder length=0.8083900654294837 radius=0.027828141337028135; visual cylinder length=0.8083900654294837 radius=0.027828141337028135
- added link 39, mass 0.001966705087677275; collision cylinder length=0.8083900654294837 radius=0.027828141337028135; visual cylinder length=0.8083900654294837 radius=0.027828141337028135
- link 0: mass 0.12562601080153418 -> 0.013499287436746527; geometry collision cylinder length=0.8406222288547908 radius=0.07149572114075056; visual cylinder length=0.8406222288547908 radius=0.07149572114075056
- link 11: mass 0.023047021486861805 -> 0.015105155920040988; geometry collision cylinder length=0.9406222288547907 radius=0.07149572114075056; visual cylinder length=0.9406222288547907 radius=0.07149572114075056
Joints:
- removed joint 12_to_0
- removed joint 23_to_0
- removed joint 24_to_0
- added joint 111_to_0: type revolute, parent 0, child 111, origin xyz=0.0 0.0 0.7895288945265722 rpy=9.471681097504312 5.511609147463753 1.433277601869214, axis 0 0 1, limit lower=3.1415 upper=-3.1415 effort=1 velocity=1
- added joint 121_to_0: type revolute, parent 0, child 121, origin xyz=0.0 0.0 0.7895288945265722 rpy=12.628908130005751 5.511609147463753 1.433277601869214, axis 0 0 1, limit lower=3.1415 upper=-3.1415 effort=1 velocity=1
- added joint 212_to_111: type revolute, parent 111, child 212, origin xyz=0.0 0.0 0.7995288945265722 rpy=6.3144540650028755 5.511609147463753 2.0615961325871726, axis 0 0 1, limit lower=3.1415 upper=-3.1415 effort=1 velocity=1
- added joint 215_to_111: type revolute, parent 111, child 215, origin xyz=0.0 0.0 0.7995288945265722 rpy=9.471681097504312 5.511609147463753 2.0615961325871726, axis 0 0 1, limit lower=3.1415 upper=-3.1415 effort=1 velocity=1
- added joint 218_to_111: type revolute, parent 111, child 218, origin xyz=0.0 0.0 0.7995288945265722 rpy=12.628908130005751 5.511609147463753 2.0615961325871726, axis 0 0 1, limit lower=3.1415 upper=-3.1415 effort=1 velocity=1
- added joint 222_to_121: type revolute, parent 121, child 222, origin xyz=0.0 0.0 0.7995288945265722 rpy=6.3144540650028755 5.511609147463753 2.0615961325871726, axis 0 0 1, limit lower=3.1415 upper=-3.1415 effort=1 velocity=1
- added joint 225_to_121: type revolute, parent 121, child 225, origin xyz=0.0 0.0 0.7995288945265722 rpy=9.471681097504312 5.511609147463753 2.0615961325871726, axis 0 0 1, limit lower=3.1415 upper=-3.1415 effort=1 velocity=1
- added joint 228_to_121: type revolute, parent 121, child 228, origin xyz=0.0 0.0 0.7995288945265722 rpy=12.628908130005751 5.511609147463753 2.0615961325871726, axis 0 0 1, limit lower=3.1415 upper=-3.1415 effort=1 velocity=1
- added joint 22_to_11: type revolute, parent 11, child 22, origin xyz=0.0 0.0 0.7995288945265722 rpy=6.3144540650028755 5.511609147463753 2.0615961325871726, axis 0 0 1, limit lower=3.1415 upper=-3.1415 effort=1 velocity=1
- added joint 25_to_11: type revolute, parent 11, child 25, origin xyz=0.0 0.0 0.7995288945265722 rpy=9.471681097504312 5.511609147463753 2.0615961325871726, axis 0 0 1, limit lower=3.1415 upper=-3.1415 effort=1 velocity=1
- added joint 28_to_11: type revolute, parent 11, child 28, origin xyz=0.0 0.0 0.7995288945265722 rpy=12.628908130005751 5.511609147463753 2.0615961325871726, axis 0 0 1, limit lower=3.1415 upper=-3.1415 effort=1 velocity=1
- added joint 310_to_28: type revolute, parent 28, child 310, origin xyz=0.0 0.0 0.7003547719575918 rpy=13.668942813438246 4.394555394056533 0.7417683914172665, axis 1 0 0, limit lower=3.1415 upper=-3.1415 effort=1 velocity=1
- added joint 313_to_212: type revolute, parent 212, child 313, origin xyz=0.0 0.0 0.7003547719575918 rpy=9.112628542292164 4.394555394056533 0.7417683914172665, axis 1 0 0, limit lower=3.1415 upper=-3.1415 effort=1 velocity=1
- added joint 314_to_212: type revolute, parent 212, child 314, origin xyz=0.0 0.0 0.7003547719575918 rpy=13.668942813438246 4.394555394056533 0.7417683914172665, axis 1 0 0, limit lower=3.1415 upper=-3.1415 effort=1 velocity=1
- added joint 316_to_215: type revolute, parent 215, child 316, origin xyz=0.0 0.0 0.7003547719575918 rpy=9.112628542292164 4.394555394056533 0.7417683914172665, axis 1 0 0, limit lower=3.1415 upper=-3.1415 effort=1 velocity=1
- added joint 317_to_215: type revolute, parent 215, child 317, origin xyz=0.0 0.0 0.7003547719575918 rpy=13.668942813438246 4.394555394056533 0.7417683914172665, axis 1 0 0, limit lower=3.1415 upper=-3.1415 effort=1 velocity=1
- added joint 319_to_218: type revolute, parent 218, child 319, origin xyz=0.0 0.0 0.7003547719575918 rpy=9.112628542292164 4.394555394056533 0.7417683914172665, axis 1 0 0, limit lower=3.1415 upper=-3.1415 effort=1 velocity=1
- added joint 320_to_218: type revolute, parent 218, child 320, origin xyz=0.0 0.0 0.7003547719575918 rpy=13.668942813438246 4.394555394056533 0.7417683914172665, axis 1 0 0, limit lower=3.1415 upper=-3.1415 effort=1 velocity=1
- added joint 323_to_222: type revolute, parent 222, child 323, origin xyz=0.0 0.0 0.7003547719575918 rpy=9.112628542292164 4.394555394056533 0.7417683914172665, axis 1 0 0, limit lower=3.1415 upper=-3.1415 effort=1 velocity=1
- added joint 324_to_222: type revolute, parent 222, child 324, origin xyz=0.0 0.0 0.7003547719575918 rpy=13.668942813438246 4.394555394056533 0.7417683914172665, axis 1 0 0, limit lower=3.1415 upper=-3.1415 effort=1 velocity=1
- added joint 326_to_225: type revolute, parent 225, child 326, origin xyz=0.0 0.0 0.7003547719575918 rpy=9.112628542292164 4.394555394056533 0.7417683914172665, axis 1 0 0, limit lower=3.1415 upper=-3.1415 effort=1 velocity=1
- added joint 327_to_225: type revolute, parent 225, child 327, origin xyz=0.0 0.0 0.7003547719575918 rpy=13.668942813438246 4.394555394056533 0.7417683914172665, axis 1 0 0, limit lower=3.1415 upper=-3.1415 effort=1 velocity=1
- added joint 329_to_228: type revolute, parent 228, child 329, origin xyz=0.0 0.0 0.7003547719575918 rpy=9.112628542292164 4.394555394056533 0.7417683914172665, axis 1 0 0, limit lower=3.1415 upper=-3.1415 effort=1 velocity=1
- added joint 330_to_228: type revolute, parent 228, child 330, origin xyz=0.0 0.0 0.7003547719575918 rpy=13.668942813438246 4.394555394056533 0.7417683914172665, axis 1 0 0, limit lower=3.1415 upper=-3.1415 effort=1 velocity=1
- added joint 33_to_22: type revolute, parent 22, child 33, origin xyz=0.0 0.0 0.7003547719575918 rpy=9.112628542292164 4.394555394056533 0.7417683914172665, axis 1 0 0, limit lower=3.1415 upper=-3.1415 effort=1 velocity=1
- added joint 34_to_22: type revolute, parent 22, child 34, origin xyz=0.0 0.0 0.7003547719575918 rpy=13.668942813438246 4.394555394056533 0.7417683914172665, axis 1 0 0, limit lower=3.1415 upper=-3.1415 effort=1 velocity=1
- added joint 36_to_25: type revolute, parent 25, child 36, origin xyz=0.0 0.0 0.7003547719575918 rpy=9.112628542292164 4.394555394056533 0.7417683914172665, axis 1 0 0, limit lower=3.1415 upper=-3.1415 effort=1 velocity=1
- added joint 37_to_25: type revolute, parent 25, child 37, origin xyz=0.0 0.0 0.7003547719575918 rpy=13.668942813438246 4.394555394056533 0.7417683914172665, axis 1 0 0, limit lower=3.1415 upper=-3.1415 effort=1 velocity=1
- added joint 39_to_28: type revolute, parent 28, child 39, origin xyz=0.0 0.0 0.7003547719575918 rpy=9.112628542292164 4.394555394056533 0.7417683914172665, axis 1 0 0, limit lower=3.1415 upper=-3.1415 effort=1 velocity=1
- joint 11_to_0: origin xyz=0.0 0.0 0.6110374662090388 rpy=4.591812931101253 6.282556988648868 0.7699242783357677 -> xyz=0.0 0.0 0.7895288945265722 rpy=6.3144540650028755 5.511609147463753 1.433277601869214
