Commit message: creature moved

File: temp0.urdf (robot description, URDF)
Before this commit: robot pepe, 2 links, 1 joints
Links:
- removed link 11
- link 0: mass 0.4447882402008654 -> 1.5747714322078803; geometry collision cylinder length=1.5393431907962147 radius=0.5706451099751567; visual cylinder length=1.5393431907962147 radius=0.5706451099751567
Joints:
- removed joint 11_to_0

File: temp1.urdf (robot description, URDF)
Before this commit: robot pepe, 1 links, 0 joints
Links:
- added link 11, mass 0.5371064366187085; collision cylinder length=1.4351199875806484 radius=0.34515258914233515; visual cylinder length=1.4351199875806484 radius=0.34515258914233515
- added link 12, mass 0.5371064366187085; collision cylinder length=1.4351199875806484 radius=0.34515258914233515; visual cylinder length=1.4351199875806484 radius=0.34515258914233515
- added link 13, mass 0.5371064366187085; collision cylinder length=1.4351199875806484 radius=0.34515258914233515; visual cylinder length=1.4351199875806484 radius=0.34515258914233515
- link 0: mass 1.651074374887958 -> 0.2375541786682687; geometry collision cylinder length=0.47657516367814656 radius=0.39832787362303057; visual cylinder length=0.47657516367814656 radius=0.39832787362303057
Joints:
- added joint 11_to_0: type revolute, parent 0, child 11, origin xyz=0.013092037684104607 0.4791579600190232 0.9999 rpy=6.957516219685191 1.6031622255808835 3.9863475536832564, axis 0 0 1, limit lower=3.1415 upper=-3.1415 effort=1 velocity=1
- added joint 12_to_0: type revolute, parent 0, child 12, origin xyz=0.013092037684104607 0.4791579600190232 0.9999 rpy=10.436274329527787 1.6031622255808835 3.9863475536832564, axis 0 0 1, limit lower=3.1415 upper=-3.1415 effort=1 velocity=1
- added joint 13_to_0: type revolute, parent 0, child 13, origin xyz=0.013092037684104607 0.4791579600190232 0.9999 rpy=13.915032439370382 1.6031622255808835 3.9863475536832564, axis 0 0 1, limit lower=3.1415 upper=-3.1415 effort=1 velocity=1

File: temp10.urdf (robot description, URDF)
Before this commit: robot pepe, 4 links, 3 joints
Links:
- removed link 11
- removed link 12
- removed link 13
- link 0: mass 0.017228056813158723 -> 0.9925645147254278; geometry collision cylinder length=0.7827782332107138 radius=0.6353090846796617; visual cylinder length=0.7827782332107138 radius=0.6353090846796617
Joints:
- removed joint 11_to_0
- removed joint 12_to_0
- removed joint 13_to_0

File: temp11.urdf (robot description, URDF)
Before this commit: robot pepe, 3 links, 2 joints
Links:
- removed link 12
- link 0: mass 6.281300540076709 -> 0.17978278050194482; geometry collision cylinder length=1.9942607892580932 radius=0.16939794399457853; visual cylinder length=1.9942607892580932 radius=0.16939794399457853
- link 11: mass 4.8509569313622345 -> 0.06312530083364862; geometry collision cylinder length=1.028297201737979 radius=0.13978721970475871; visual cylinder length=1.028297201737979 radius=0.13978721970475871
Joints:
- removed joint 12_to_0
- joint 11_to_0: axis 0 0 1 -> 1 0 0; origin xyz=0.6288798798451473 0.21263318293317526 0.30695240406001423 rpy=4.536694574069128 5.441986758342813 5.552140457765634 -> xyz=0.9274683407053369 0.2336947875517995 0.3539347662641653 rpy=6.528734028025818 6.282556988648868 2.530502266948649

File: temp2.urdf (robot description, URDF)
Before this commit: robot pepe, 1 links, 0 joints
Links:
- added link 11, mass 0.004273567102552457; collision cylinder length=0.25905983768236474 radius=0.07246366287879047; visual cylinder length=0.25905983768236474 radius=0.07246366287879047
- link 0: mass 0.8767528697274423 -> 1.5747714322078803; geometry collision cylinder length=1.5393431907962147 radius=0.5706451099751567; visual cylinder length=1.5393431907962147 radius=0.5706451099751567
Joints:
- added joint 11_to_0: type revolute, parent 0, child 11, origin xyz=0.20875914034680187 0.49110837623561154 0.8877718433181635 rpy=3.912101849663146 0.024033328500454053 0.7565086088087307, axis 0 0 1, limit lower=3.1415 upper=-3.1415 effort=1 velocity=1

File: temp3.urdf (robot description, URDF)
Before this commit: robot pepe, 1 links, 0 joints
Links:
- added link 11, mass 0.010502503495838894; collision cylinder length=1.4103494861924255 radius=0.04868644998176164; visual cylinder length=1.4103494861924255 radius=0.04868644998176164
- added link 22, mass 0.91716554023611; collision cylinder length=1.295877378317102 radius=0.47464288367026597; visual cylinder length=1.295877378317102 radius=0.47464288367026597
- link 0: mass 6.281300540076709 -> 0.0207233969095683; geometry collision cylinder length=0.22708795576946345 radius=0.1704348825760488; visual cylinder length=0.22708795576946345 radius=0.1704348825760488
Joints:
- added joint 11_to_0: type revolute, parent 0, child 11, origin xyz=0.22566846990232847 0.8369671024592621 0.48585498233183066 rpy=5.157333295744659 6.282556988648868 6.282556988648868, axis 0 1 0, limit lower=3.1415 upper=-3.1415 effort=1 velocity=1
- added joint 22_to_0: type revolute, parent 0, child 22, origin xyz=0.2538285945708213 0.2333768945901622 0.01267128401551465 rpy=18.31639586105737 3.9333437046616435 4.537356693450489, axis 1 0 0, limit lower=3.1415 upper=-3.1415 effort=1 velocity=1

File: temp4.urdf (robot description, URDF)
Before this commit: robot pepe, 10 links, 9 joints
Links:
- removed link 11
- removed link 14
- removed link 17
- removed link 22
- removed link 23
- removed link 25
- removed link 26
- removed link 28
- removed link 29
- link 0: mass 4.8509569313622345 -> 0.4622546554064389; geometry collision cylinder length=1.2351199875806484 radius=0.34515258914233515; visual cylinder length=1.2351199875806484 radius=0.34515258914233515
Joints:
- removed joint 11_to_0
- removed joint 14_to_0
- removed joint 17_to_0
- removed joint 22_to_11
- removed joint 23_to_11
- removed joint 25_to_14
- removed joint 26_to_14
- removed joint 28_to_17
- removed joint 29_to_17

File: temp5.urdf (robot description, URDF)
Before this commit: robot pepe, 3 links, 2 joints
Links:
- link 0: mass 4.8509569313622345 -> 0.058890981107942074; geometry collision cylinder length=0.47657516367814656 radius=0.19832787362303061; visual cylinder length=0.47657516367814656 radius=0.19832787362303061
- link 11: mass 0.00015899238161076818 -> 2.1750580493753975; geometry collision cylinder length=1.5393431907962147 radius=0.6706451099751567; visual cylinder length=1.5393431907962147 radius=0.6706451099751567
- link 12: mass 0.00015899238161076818 -> 2.1750580493753975; geometry collision cylinder length=1.5393431907962147 radius=0.6706451099751567; visual cylinder length=1.5393431907962147 radius=0.6706451099751567
Joints:
- joint 11_to_0: origin xyz=0.6460249959333256 0.7977241153738953 0.11796893835155542 rpy=4.880045374580523 2.8198353222488572 0.10982749423898357 -> xyz=0.8736226382061546 0.7804747334818708 0.9999 rpy=6.607168032624262 6.282556988648868 2.431444931381071
- joint 12_to_0: origin xyz=0.6460249959333256 0.7977241153738953 0.11796893835155542 rpy=7.320068061870785 2.8198353222488572 0.10982749423898357 -> xyz=0.8736226382061546 0.7804747334818708 0.9999 rpy=9.910752048936393 6.282556988648868 2.431444931381071

File: temp6.urdf (robot description, URDF)
Before this commit: robot pepe, 4 links, 3 joints
Links:
- removed link 12
- removed link 13
- link 0: mass 5.646653933224324 -> 0.40537590985467736; geometry collision cylinder length=1.039763113429477 radius=0.35227905988919916; visual cylinder length=1.039763113429477 radius=0.35227905988919916
- link 11: mass 0.666736660016075 -> 1.8001805889964049; geometry collision cylinder length=1.9998 radius=0.5352908488159872; visual cylinder length=1.9998 radius=0.5352908488159872
Joints:
- removed joint 12_to_0
- removed joint 13_to_0
- joint 11_to_0: axis 1 0 0 -> 0 0 1; origin xyz=0.4003180817346731 0.06349376569629328 0.8419032451969989 rpy=10.076326353719763 5.508166182377774 0.7793229481478409 -> xyz=0.3458675587015642 0.5012319438492308 0.2032645901093748 rpy=11.686798263636996 6.282556988648868 0.9819415266837115

File: temp7.urdf (robot description, URDF)
Before this commit: robot pepe, 1 links, 0 joints
Links:
- added link 11, mass 0.06425666732148974; collision cylinder length=1.1748686165879532 radius=0.13194395890596244; visual cylinder length=1.1748686165879532 radius=0.13194395890596244
- added link 12, mass 0.06425666732148974; collision cylinder length=1.1748686165879532 radius=0.13194395890596244; visual cylinder length=1.1748686165879532 radius=0.13194395890596244
- added link 13, mass 0.06425666732148974; collision cylinder length=1.1748686165879532 radius=0.13194395890596244; visual cylinder length=1.1748686165879532 radius=0.13194395890596244
- link 0: mass 4.982139687530963 -> 0.011154690088598603; geometry collision cylinder length=0.8242377192703865 radius=0.0656338039526092; visual cylinder length=0.8242377192703865 radius=0.0656338039526092
Joints:
- added joint 11_to_0: type revolute, parent 0, child 11, origin xyz=0.07374001551327147 0.2739473156868729 0.6667025459214211 rpy=12.480308541222044 1.4673991856423787 5.961105602087462, axis 0 1 0, limit lower=3.1415 upper=-3.1415 effort=1 velocity=1
- added joint 12_to_0: type revolute, parent 0, child 12, origin xyz=0.07374001551327147 0.2739473156868729 0.6667025459214211 rpy=18.720462811833066 1.4673991856423787 5.961105602087462, axis 0 1 0, limit lower=3.1415 upper=-3.1415 effort=1 velocity=1
- added joint 13_to_0: type revolute, parent 0, child 13, origin xyz=0.07374001551327147 0.2739473156868729 0.6667025459214211 rpy=24.960617082444088 1.4673991856423787 5.961105602087462, axis 0 1 0, limit lower=3.1415 upper=-3.1415 effort=1 velocity=1

File: temp8.urdf (robot description, URDF)
Before this commit: robot pepe, 1 links, 0 joints
Links:
- added link 11, mass 1.2461649529119203; collision cylinder length=0.9827782332107138 radius=0.6353090846796617; visual cylinder length=0.9827782332107138 radius=0.6353090846796617
- added link 12, mass 1.2461649529119203; collision cylinder length=0.9827782332107138 radius=0.6353090846796617; visual cylinder length=0.9827782332107138 radius=0.6353090846796617
- added link 13, mass 1.2461649529119203; collision cylinder length=0.9827782332107138 radius=0.6353090846796617; visual cylinder length=0.9827782332107138 radius=0.6353090846796617
- link 0: mass 2.231598294664083 -> 0.1678336337945813; geometry collision cylinder length=1.1739940931651733 radius=0.2133200155056895; visual cylinder length=1.1739940931651733 radius=0.2133200155056895
Joints:
- added joint 11_to_0: type revolute, parent 0, child 11, origin xyz=0.48338204848938504 0.2374669109417115 0.8576115813268254 rpy=8.681631304303965 0.11156870956857395 1.7593560540737883, axis 0 0 1, limit lower=3.1415 upper=-3.1415 effort=1 velocity=1
- added joint 12_to_0: type revolute, parent 0, child 12, origin xyz=0.48338204848938504 0.2374669109417115 0.8576115813268254 rpy=13.022446956455948 0.11156870956857395 1.7593560540737883, axis 0 0 1, limit lower=3.1415 upper=-3.1415 effort=1 velocity=1
- added joint 13_to_0: type revolute, parent 0, child 13, origin xyz=0.48338204848938504 0.2374669109417115 0.8576115813268254 rpy=17.36326260860793 0.11156870956857395 1.7593560540737883, axis 0 0 1, limit lower=3.1415 upper=-3.1415 effort=1 velocity=1

File: temp9.urdf (robot description, URDF)
Before this commit: robot pepe, 2 links, 1 joints
Links:
- added link 12, mass 0.5810690302092903; collision cylinder length=0.8073689846538772 radius=0.47863328536728944; visual cylinder length=0.8073689846538772 radius=0.47863328536728944
- added link 13, mass 0.5810690302092903; collision cylinder length=0.8073689846538772 radius=0.47863328536728944; visual cylinder length=0.8073689846538772 radius=0.47863328536728944
- link 0: mass 6.281300540076709 -> 0.2375541786682687; geometry collision cylinder length=0.47657516367814656 radius=0.39832787362303057; visual cylinder length=0.47657516367814656 radius=0.39832787362303057
- link 11: mass 6.281300540076709 -> 0.5810690302092903; geometry collision cylinder length=0.8073689846538772 radius=0.47863328536728944; visual cylinder length=0.8073689846538772 radius=0.47863328536728944
Joints:
- added joint 12_to_0: type revolute, parent 0, child 12, origin xyz=0.8546945632695275 0.3560870915853548 0.9999 rpy=17.615755185976894 1.8546724403422652 1.7009194973071655, axis 0 1 0, limit lower=3.1415 upper=-3.1415 effort=1 velocity=1
- added joint 13_to_0: type revolute, parent 0, child 13, origin xyz=0.8546945632695275 0.3560870915853548 0.9999 rpy=23.487673581302527 1.8546724403422652 1.7009194973071655, axis 0 1 0, limit lower=3.1415 upper=-3.1415 effort=1 velocity=1
- joint 11_to_0: axis 0 0 1 -> 0 1 0; origin xyz=0.034281998243213097 0.9970823748954981 0.7107158982434543 rpy=10.727363753556237 3.299445189783009 2.647693178317944 -> xyz=0.8546945632695275 0.3560870915853548 0.9999 rpy=11.743836790651264 1.8546724403422652 1.7009194973071655

File: test.urdf (robot description, URDF)
Before this commit: robot pepe, 9 links, 8 joints
Links:
- removed link 15
- removed link 24
- removed link 26
- removed link 27
- removed link 28
- link 0: mass 0.0006266931023623138 -> 0.0035393178252391836; geometry collision cylinder length=0.22708795576946345 radius=0.0704348825760488; visual cylinder length=0.22708795576946345 radius=0.0704348825760488
- link 11: mass 0.036815199820519305 -> 3.256053281005642; geometry collision cylinder length=1.2889579130614948 radius=0.8967088305527183; visual cylinder length=1.2889579130614948 radius=0.8967088305527183
- link 22: mass 2.109157485313338 -> 4.030376295646057; geometry collision cylinder length=1.2831652401613243 radius=0.9999; visual cylinder length=1.2831652401613243 radius=0.9999
- link 23: mass 2.109157485313338 -> 4.030376295646057; geometry collision cylinder length=1.2831652401613243 radius=0.9999; visual cylinder length=1.2831652401613243 radius=0.9999
Joints:
- removed joint 15_to_0
- removed joint 24_to_11
- removed joint 26_to_15
- removed joint 27_to_15
- removed joint 28_to_15
- joint 11_to_0: axis 1 0 0 -> 0 1 0; origin xyz=0.9211911784477138 0.9999 0.22097220481951255 rpy=6.686760282733851 5.507066050751844 2.4867577634447517 -> xyz=0.21517117883011172 0.8602392471751297 0.2948748084169591 rpy=9.971405700062027 2.233838326512593 4.399607301567375
- joint 22_to_11: axis 0 1 0 -> 0 0 1; origin xyz=0.5723003634453724 0.7343359490418989 0.004789470228331982 rpy=8.582294283103815 6.022524202784673 3.2204442206050974 -> xyz=0.8757516180870302 0.3802844087754167 0.7207534385083066 rpy=8.925674400481595 1.4185095832482375 3.514743627616129
- joint 23_to_11: axis 0 1 0 -> 0 0 1; origin xyz=0.5723003634453724 0.7343359490418989 0.004789470228331982 rpy=12.873441424655724 6.022524202784673 3.2204442206050974 -> xyz=0.8757516180870302 0.3802844087754167 0.7207534385083066 rpy=13.388511600722392 1.4185095832482375 3.514743627616129
