Commit message: logging implemented, ready for experimentation

File: temp0.urdf (robot description, URDF)
Before this commit: robot pepe, 5 links, 4 joints
Links:
- removed link 22
- removed link 23
- removed link 24
- link 0: mass 0.03282971740437995 -> 0.01511010110913815; geometry collision cylinder length=0.18572363406517922 radius=0.16092560939485884; visual cylinder length=0.18572363406517922 radius=0.16092560939485884
- link 11: mass 0.05504305957367886 -> 0.01511010110913815; geometry collision cylinder length=0.18572363406517922 radius=0.16092560939485884; visual cylinder length=0.18572363406517922 radius=0.16092560939485884
Joints:
- removed joint 22_to_11
- removed joint 23_to_11
- removed joint 24_to_11
- joint 11_to_0: axis 0 1 0 -> 0 0 1; origin xyz=0.0 0.0 0.6074492098211774 rpy=10.574162790228621 1.6754903303533237 1.0066778357037864 -> xyz=0.0 0.0 0.15786508895540233 rpy=8.174625539400152 5.446621470180249 4.900426046421999

File: temp1.urdf (robot description, URDF)
Before this commit: robot pepe, 10 links, 9 joints
Links:
- removed link 14
- removed link 17
- removed link 22
- removed link 25
- removed link 28
- removed link 33
- removed link 36
- removed link 39
- added link 12, mass 0.12562601080153418; collision cylinder length=0.9999 radius=0.19998000000000002; visual cylinder length=0.9999 radius=0.19998000000000002
- added link 13, mass 0.12562601080153418; collision cylinder length=0.9999 radius=0.19998000000000002; visual cylinder length=0.9999 radius=0.19998000000000002
- added link 24, mass 0.01511010110913815; collision cylinder length=0.18572363406517922 radius=0.16092560939485884; visual cylinder length=0.18572363406517922 radius=0.16092560939485884
- link 0: mass 0.05109617055670747 -> 0.1146116058470627; geometry collision cylinder length=0.9999 radius=0.19101218751194338; visual cylinder length=0.9999 radius=0.19101218751194338
- link 11: mass 0.03282971740437995 -> 0.12562601080153418; geometry collision cylinder length=0.9999 radius=0.19998000000000002; visual cylinder length=0.9999 radius=0.19998000000000002
Joints:
- removed joint 14_to_0
- removed joint 17_to_0
- removed joint 22_to_11
- removed joint 25_to_14
- removed joint 28_to_17
- removed joint 33_to_11
- removed joint 36_to_14
- removed joint 39_to_17
- added joint 12_to_0: type revolute, parent 0, child 12, origin xyz=0.0 0.0 0.849915 rpy=18.847670965946605 5.337894333820069 6.282556988648868, axis 0 0 1, limit lower=3.1415 upper=-3.1415 effort=1 velocity=1
- added joint 13_to_0: type revolute, parent 0, child 13, origin xyz=0.0 0.0 0.849915 rpy=25.130227954595473 5.337894333820069 6.282556988648868, axis 0 0 1, limit lower=3.1415 upper=-3.1415 effort=1 velocity=1
- added joint 24_to_0: type revolute, parent 0, child 24, origin xyz=0.0 0.0 0.2392827255488844 rpy=20.43656384850038 5.446621470180249 4.900426046421999, axis 0 0 1, limit lower=3.1415 upper=-3.1415 effort=1 velocity=1
- joint 11_to_0: origin xyz=0.0 0.0 0.7245288945265721 rpy=7.571091126438793 6.282556988648868 2.0615961325871726 -> xyz=0.0 0.0 0.849915 rpy=12.565113977297736 5.337894333820069 6.282556988648868

File: temp2.urdf (robot description, URDF)
Before this commit: robot pepe, 2 links, 1 joints
Links:
- added link 12, mass 0.12562601080153418; collision cylinder length=0.9999 radius=0.19998000000000002; visual cylinder length=0.9999 radius=0.19998000000000002
- added link 13, mass 0.12562601080153418; collision cylinder length=0.9999 radius=0.19998000000000002; visual cylinder length=0.9999 radius=0.19998000000000002
- link 0: mass 0.05504305957367886 -> 0.1146116058470627; geometry collision cylinder length=0.9999 radius=0.19101218751194338; visual cylinder length=0.9999 radius=0.19101218751194338
- link 11: mass 0.05504305957367886 -> 0.12562601080153418; geometry collision cylinder length=0.9999 radius=0.19998000000000002; visual cylinder length=0.9999 radius=0.19998000000000002
Joints:
- added joint 12_to_0: type revolute, parent 0, child 12, origin xyz=0.0 0.0 0.849915 rpy=17.012340233558895 5.337894333820069 6.282556988648868, axis 0 0 1, limit lower=3.1415 upper=-3.1415 effort=1 velocity=1
- added joint 13_to_0: type revolute, parent 0, child 13, origin xyz=0.0 0.0 0.849915 rpy=22.683120311411862 5.337894333820069 6.282556988648868, axis 0 0 1, limit lower=3.1415 upper=-3.1415 effort=1 velocity=1
- joint 11_to_0: axis 0 1 0 -> 0 0 1; origin xyz=0.0 0.0 0.5931719185271249 rpy=10.574162790228621 1.0471717996353653 1.0066778357037864 -> xyz=0.0 0.0 0.849915 rpy=11.341560155705931 5.337894333820069 6.282556988648868

File: temp3.urdf (robot description, URDF)
Before this commit: robot pepe, 5 links, 4 joints
Links:
- link 0: mass 0.03282971740437995 -> 0.12562601080153418; geometry collision cylinder length=0.9999 radius=0.19998000000000002; visual cylinder length=0.9999 radius=0.19998000000000002
- link 11: mass 0.05504305957367886 -> 0.01511010110913815; geometry collision cylinder length=0.18572363406517922 radius=0.16092560939485884; visual cylinder length=0.18572363406517922 radius=0.16092560939485884
- link 22: mass 0.036735124170639864 -> 0.1146116058470627; geometry collision cylinder length=0.9999 radius=0.19101218751194338; visual cylinder length=0.9999 radius=0.19101218751194338
- link 23: mass 0.036735124170639864 -> 0.1146116058470627; geometry collision cylinder length=0.9999 radius=0.19101218751194338; visual cylinder length=0.9999 radius=0.19101218751194338
- link 24: mass 0.036735124170639864 -> 0.1146116058470627; geometry collision cylinder length=0.9999 radius=0.19101218751194338; visual cylinder length=0.9999 radius=0.19101218751194338
Joints:
- joint 11_to_0: axis 0 1 0 -> 0 0 1; origin xyz=0.0 0.0 0.6074492098211774 rpy=10.574162790228621 1.0471717996353653 1.0066778357037864 -> xyz=0.0 0.0 0.2392827255488844 rpy=8.174625539400152 5.446621470180249 4.900426046421999
- joint 22_to_11: origin xyz=0.0 0.0 0.7752516032325196 rpy=7.571091126438793 6.282556988648868 2.0615961325871726 -> xyz=0.0 0.0 0.7684973634065179 rpy=11.341560155705931 5.337894333820069 6.282556988648868
- joint 23_to_11: origin xyz=0.0 0.0 0.7752516032325196 rpy=11.356636689658188 6.282556988648868 2.0615961325871726 -> xyz=0.0 0.0 0.7684973634065179 rpy=17.012340233558895 5.337894333820069 6.282556988648868
- joint 24_to_11: origin xyz=0.0 0.0 0.7752516032325196 rpy=15.142182252877586 6.282556988648868 2.0615961325871726 -> xyz=0.0 0.0 0.7684973634065179 rpy=22.683120311411862 5.337894333820069 6.282556988648868

File: temp4.urdf (robot description, URDF)
Before this commit: robot pepe, 3 links, 2 joints
Links:
- removed link 22
- added link 12, mass 0.12562601080153418; collision cylinder length=0.9999 radius=0.19998000000000002; visual cylinder length=0.9999 radius=0.19998000000000002
- added link 13, mass 0.12562601080153418; collision cylinder length=0.9999 radius=0.19998000000000002; visual cylinder length=0.9999 radius=0.19998000000000002
- added link 24, mass 0.023245899864742566; collision cylinder length=0.2857236340651792 radius=0.16092560939485884; visual cylinder length=0.2857236340651792 radius=0.16092560939485884
- added link 35, mass 0.001740575968251717; collision cylinder length=0.1769882521642463 radius=0.055949902615489; visual cylinder length=0.1769882521642463 radius=0.055949902615489
- added link 36, mass 0.001740575968251717; collision cylinder length=0.1769882521642463 radius=0.055949902615489; visual cylinder length=0.1769882521642463 radius=0.055949902615489
- added link 37, mass 0.001740575968251717; collision cylinder length=0.1769882521642463 radius=0.055949902615489; visual cylinder length=0.1769882521642463 radius=0.055949902615489
- link 0: mass 0.05504305957367886 -> 0.1146116058470627; geometry collision cylinder length=0.9999 radius=0.19101218751194338; visual cylinder length=0.9999 radius=0.19101218751194338
- link 11: mass 0.06293058748528338 -> 0.12562601080153418; geometry collision cylinder length=0.9999 radius=0.19998000000000002; visual cylinder length=0.9999 radius=0.19998000000000002
Joints:
- removed joint 22_to_11
- added joint 12_to_0: type revolute, parent 0, child 12, origin xyz=0.0 0.0 0.849915 rpy=17.012340233558895 5.337894333820069 6.282556988648868, axis 0 0 1, limit lower=3.1415 upper=-3.1415 effort=1 velocity=1
- added joint 13_to_0: type revolute, parent 0, child 13, origin xyz=0.0 0.0 0.849915 rpy=22.683120311411862 5.337894333820069 6.282556988648868, axis 0 0 1, limit lower=3.1415 upper=-3.1415 effort=1 velocity=1
- added joint 24_to_0: type revolute, parent 0, child 24, origin xyz=0.0 0.0 0.3142827255488844 rpy=20.43656384850038 5.446621470180249 4.900426046421999, axis 0 0 1, limit lower=3.1415 upper=-3.1415 effort=1 velocity=1
- added joint 35_to_0: type revolute, parent 0, child 35, origin xyz=0.0 0.0 0.23273118912318475 rpy=36.24561496854278 1.5451808687618354 1.4106858308233514, axis 0 0 1, limit lower=3.1415 upper=-3.1415 effort=1 velocity=1
- added joint 36_to_0: type revolute, parent 0, child 36, origin xyz=0.0 0.0 0.23273118912318475 rpy=42.28655079663324 1.5451808687618354 1.4106858308233514, axis 0 0 1, limit lower=3.1415 upper=-3.1415 effort=1 velocity=1
- added joint 37_to_0: type revolute, parent 0, child 37, origin xyz=0.0 0.0 0.23273118912318475 rpy=48.327486624723704 1.5451808687618354 1.4106858308233514, axis 0 0 1, limit lower=3.1415 upper=-3.1415 effort=1 velocity=1
- joint 11_to_0: axis 0 1 0 -> 0 0 1; origin xyz=0.0 0.0 0.6681719185271249 rpy=9.317525728792704 1.0471717996353653 1.0066778357037864 -> xyz=0.0 0.0 0.849915 rpy=11.341560155705931 5.337894333820069 6.282556988648868

File: temp5.urdf (robot description, URDF)
Before this commit: robot pepe, 10 links, 9 joints
Links:
- removed link 14
- removed link 17
- removed link 22
- removed link 25
- removed link 28
- removed link 33
- removed link 36
- removed link 39
- added link 12, mass 0.12562601080153418; collision cylinder length=0.9999 radius=0.19998000000000002; visual cylinder length=0.9999 radius=0.19998000000000002
- added link 13, mass 0.12562601080153418; collision cylinder length=0.9999 radius=0.19998000000000002; visual cylinder length=0.9999 radius=0.19998000000000002
- added link 24, mass 0.01511010110913815; collision cylinder length=0.18572363406517922 radius=0.16092560939485884; visual cylinder length=0.18572363406517922 radius=0.16092560939485884
- link 0: mass 0.05504305957367886 -> 0.1146116058470627; geometry collision cylinder length=0.9999 radius=0.19101218751194338; visual cylinder length=0.9999 radius=0.19101218751194338
- link 11: mass 0.03282971740437995 -> 0.12562601080153418; geometry collision cylinder length=0.9999 radius=0.19998000000000002; visual cylinder length=0.9999 radius=0.19998000000000002
Joints:
- removed joint 14_to_0
- removed joint 17_to_0
- removed joint 22_to_11
- removed joint 25_to_14
- removed joint 28_to_17
- removed joint 33_to_11
- removed joint 36_to_14
- removed joint 39_to_17
- added joint 12_to_0: type revolute, parent 0, child 12, origin xyz=0.0 0.0 0.849915 rpy=17.012340233558895 5.337894333820069 6.282556988648868, axis 0 0 1, limit lower=3.1415 upper=-3.1415 effort=1 velocity=1
- added joint 13_to_0: type revolute, parent 0, child 13, origin xyz=0.0 0.0 0.849915 rpy=22.683120311411862 5.337894333820069 6.282556988648868, axis 0 0 1, limit lower=3.1415 upper=-3.1415 effort=1 velocity=1
- added joint 24_to_0: type revolute, parent 0, child 24, origin xyz=0.0 0.0 0.2392827255488844 rpy=20.43656384850038 6.0749400008982075 4.900426046421999, axis 0 0 1, limit lower=3.1415 upper=-3.1415 effort=1 velocity=1
- joint 11_to_0: origin xyz=0.0 0.0 0.7002516032325194 rpy=7.571091126438793 6.282556988648868 2.0615961325871726 -> xyz=0.0 0.0 0.849915 rpy=11.341560155705931 5.337894333820069 6.282556988648868

File: test.urdf (robot description, URDF)
Before this commit: robot pepe, 31 links, 30 joints
Links:
- removed link 111
- removed link 121
- removed link 212
- removed link 215
- removed link 218
- removed link 222
- removed link 225
- removed link 228
- removed link 25
- removed link 28
- removed link 313
- removed link 316
- removed link 317
- removed link 319
- removed link 320
- removed link 323
- removed link 324
- removed link 326
- removed link 327
- removed link 329
- removed link 330
- removed link 34
- removed link 36
- removed link 39
- added link 18, mass 5.0651149152824064e-05; collision cylinder length=0.13282693791763203 radius=0.011017337019195073; visual cylinder length=0.13282693791763203 radius=0.011017337019195073
- added link 211, mass 0.026814024362670986; collision cylinder length=0.44860448229249816 radius=0.1379349301151079; visual cylinder length=0.44860448229249816 radius=0.1379349301151079
- added link 213, mass 0.026814024362670986; collision cylinder length=0.44860448229249816 radius=0.1379349301151079; visual cylinder length=0.44860448229249816 radius=0.1379349301151079
- added link 24, mass 0.026814024362670986; collision cylinder length=0.44860448229249816 radius=0.1379349301151079; visual cylinder length=0.44860448229249816 radius=0.1379349301151079
- added link 26, mass 0.026814024362670986; collision cylinder length=0.44860448229249816 radius=0.1379349301151079; visual cylinder length=0.44860448229249816 radius=0.1379349301151079
- added link 29, mass 0.026814024362670986; collision cylinder length=0.44860448229249816 radius=0.1379349301151079; visual cylinder length=0.44860448229249816 radius=0.1379349301151079
- added link 312, mass 1.2517958742130715e-05; collision cylinder length=0.032826937917632026 radius=0.011017337019195073; visual cylinder length=0.032826937917632026 radius=0.011017337019195073
- added link 35, mass 1.2517958742130715e-05; collision cylinder length=0.032826937917632026 radius=0.011017337019195073; visual cylinder length=0.032826937917632026 radius=0.011017337019195073
- added link 415, mass 0.0524849787444478; collision cylinder length=0.9250295807813727 radius=0.13438932296350048; visual cylinder length=0.9250295807813727 radius=0.13438932296350048
- link 0: mass 0.013499287436746527 -> 0.03515360483035982; geometry collision cylinder length=0.44860448229249816 radius=0.15793493011510792; visual cylinder length=0.44860448229249816 radius=0.15793493011510792
- link 11: mass 0.015105155920040988 -> 5.0651149152824064e-05; geometry collision cylinder length=0.13282693791763203 radius=0.011017337019195073; visual cylinder length=0.13282693791763203 radius=0.011017337019195073
- link 22: mass 0.015105155920040988 -> 0.026814024362670986; geometry collision cylinder length=0.44860448229249816 radius=0.1379349301151079; visual cylinder length=0.44860448229249816 radius=0.1379349301151079
- link 310: mass 0.001966705087677275 -> 1.2517958742130715e-05; geometry collision cylinder length=0.032826937917632026 radius=0.011017337019195073; visual cylinder length=0.032826937917632026 radius=0.011017337019195073
- link 314: mass 0.001966705087677275 -> 1.2517958742130715e-05; geometry collision cylinder length=0.032826937917632026 radius=0.011017337019195073; visual cylinder length=0.032826937917632026 radius=0.011017337019195073
- link 33: mass 0.001966705087677275 -> 1.2517958742130715e-05; geometry collision cylinder length=0.032826937917632026 radius=0.011017337019195073; visual cylinder length=0.032826937917632026 radius=0.011017337019195073
- link 37: mass 0.001966705087677275 -> 1.2517958742130715e-05; geometry collision cylinder length=0.032826937917632026 radius=0.011017337019195073; visual cylinder length=0.032826937917632026 radius=0.011017337019195073
Joints:
- removed joint 111_to_0
- removed joint 121_to_0
- removed joint 212_to_111
- removed joint 215_to_111
- removed joint 218_to_111
- removed joint 222_to_121
- removed joint 225_to_121
- removed joint 228_to_121
- removed joint 25_to_11
- removed joint 28_to_11
- removed joint 310_to_28
- removed joint 313_to_212
- removed joint 314_to_212
- removed joint 316_to_215
- removed joint 317_to_215
- removed joint 319_to_218
- removed joint 320_to_218
- removed joint 323_to_222
- removed joint 324_to_222
- removed joint 326_to_225
- removed joint 327_to_225
- removed joint 329_to_228
- removed joint 330_to_228
- removed joint 34_to_22
- removed joint 36_to_25
- removed joint 37_to_25
- removed joint 39_to_28
- added joint 18_to_0: type revolute, parent 0, child 18, origin xyz=0.0 0.0 0.14448065166747384 rpy=12.771493493974695 1.8145901362651966 5.0096716650635065, axis 1 0 0, limit lower=3.1415 upper=-3.1415 effort=1 velocity=1
- added joint 211_to_18: type revolute, parent 18, child 211, origin xyz=0.0 0.0 0.34973605551113685 rpy=18.847670965946605 0.6760950543561008 3.8705279938633717, axis 0 0 1, limit lower=3.1415 upper=-3.1415 effort=1 velocity=1
- added joint 213_to_18: type revolute, parent 18, child 213, origin xyz=0.0 0.0 0.34973605551113685 rpy=25.130227954595473 0.6760950543561008 3.8705279938633717, axis 0 0 1, limit lower=3.1415 upper=-3.1415 effort=1 velocity=1
- added joint 24_to_11: type revolute, parent 11, child 24, origin xyz=0.0 0.0 0.34973605551113685 rpy=18.847670965946605 0.6760950543561008 3.8705279938633717, axis 0 0 1, limit lower=3.1415 upper=-3.1415 effort=1 velocity=1
- added joint 26_to_11: type revolute, parent 11, child 26, origin xyz=0.0 0.0 0.34973605551113685 rpy=25.130227954595473 0.6760950543561008 3.8705279938633717, axis 0 0 1, limit lower=3.1415 upper=-3.1415 effort=1 velocity=1
- added joint 29_to_18: type revolute, parent 18, child 29, origin xyz=0.0 0.0 0.34973605551113685 rpy=12.565113977297736 0.6760950543561008 3.8705279938633717, axis 0 0 1, limit lower=3.1415 upper=-3.1415 effort=1 velocity=1
- added joint 310_to_29: type revolute, parent 29, child 310, origin xyz=0.0 0.0 0.06948065166747383 rpy=8.51432899598313 1.8145901362651966 5.637990195781465, axis 1 0 0, limit lower=3.1415 upper=-3.1415 effort=1 velocity=1
- added joint 312_to_211: type revolute, parent 211, child 312, origin xyz=0.0 0.0 0.06948065166747383 rpy=8.51432899598313 1.8145901362651966 5.637990195781465, axis 1 0 0, limit lower=3.1415 upper=-3.1415 effort=1 velocity=1
- added joint 314_to_213: type revolute, parent 213, child 314, origin xyz=0.0 0.0 0.06948065166747383 rpy=8.51432899598313 1.8145901362651966 5.637990195781465, axis 1 0 0, limit lower=3.1415 upper=-3.1415 effort=1 velocity=1
- added joint 35_to_24: type revolute, parent 24, child 35, origin xyz=0.0 0.0 0.06948065166747383 rpy=8.51432899598313 1.8145901362651966 5.637990195781465, axis 1 0 0, limit lower=3.1415 upper=-3.1415 effort=1 velocity=1
- added joint 37_to_26: type revolute, parent 26, child 37, origin xyz=0.0 0.0 0.06948065166747383 rpy=8.51432899598313 1.8145901362651966 5.637990195781465, axis 1 0 0, limit lower=3.1415 upper=-3.1415 effort=1 velocity=1
- added joint 415_to_0: type revolute, parent 0, child 415, origin xyz=0.0 0.0 0.7386326338152793 rpy=10.66804537968895 0.018999097728681684 5.9870178031897945, axis 0 0 1, limit lower=3.1415 upper=-3.1415 effort=1 velocity=1
- joint 11_to_0: axis 0 0 1 -> 1 0 0; origin xyz=0.0 0.0 0.7895288945265722 rpy=6.3144540650028755 5.511609147463753 1.433277601869214 -> xyz=0.0 0.0 0.14448065166747384 rpy=8.51432899598313 1.8145901362651966 5.0096716650635065
- joint 22_to_11: origin xyz=0.0 0.0 0.7995288945265722 rpy=6.3144540650028755 5.511609147463753 2.0615961325871726 -> xyz=0.0 0.0 0.34973605551113685 rpy=12.565113977297736 0.6760950543561008 3.8705279938633717
- joint 33_to_22: origin xyz=0.0 0.0 0.7003547719575918 rpy=9.112628542292164 4.394555394056533 0.7417683914172665 -> xyz=0.0 0.0 0.06948065166747383 rpy=8.51432899598313 1.8145901362651966 5.637990195781465
